Commit message: dof arm added

File: urdf/so_100_arm_7dof.urdf (robot description, URDF)
Before this commit: robot so_100_arm, 9 links, 8 joints
Links:
- added link world
- link Base: geometry collision mesh filename=package://so_100_arm/models/so_100_arm_7dof/meshes/Base.STL; visual mesh filename=package://so_100_arm/models/so_100_arm_7dof/meshes/Base.STL
- link End_Servo: geometry collision mesh filename=package://so_100_arm/models/so_100_arm_7dof/meshes/End_Serv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; visual mesh filename=package://so_100_arm/models/so_100_arm_7dof/meshes/End_Serv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
- link Forearm: geometry collision mesh filename=package://so_100_arm/models/so_100_arm_7dof/meshes/Forearm.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; visual mesh filename=package://so_100_arm/models/so_100_arm_7dof/meshes/Forearm.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
- link Humeral_Elbow: geometry collision mesh filename=package://so_100_arm/models/so_100_arm_7dof/meshes/Humeral_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; visual mesh filename=package://so_100_arm/models/so_100_arm_7dof/meshes/Humeral_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
- link Shoulder_Pitch_Yaw: geometry collision mesh filename=package://so_100_arm/models/so_100_arm_7dof/meshes/Shoulder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; visual mesh filename=package://so_100_arm/models/so_100_arm_7dof/meshes/Shoulder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
- link Upper_Humeral: geometry collision mesh filename=package://so_100_arm/models/so_100_arm_7dof/meshes/Upper_Hu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; visual mesh filename=package://so_100_arm/models/so_100_arm_7dof/meshes/Upper_Hu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
- link Wrist_Roll_Yaw: geometry collision mesh filename=package://so_100_arm/models/so_100_arm_7dof/meshes/Wrist_Ro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; visual mesh filename=package://so_100_arm/models/so_100_arm_7dof/meshes/Wrist_Ro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
- link Wrist_Yaw_Pitch: geometry collision mesh filename=package://so_100_arm/models/so_100_arm_7dof/meshes/Wrist_Ya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; visual mesh filename=package://so_100_arm/models/so_100_arm_7dof/meshes/Wrist_Ya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
Joints:
- added joint world_to_base: type fixed, parent world, child base_link, origin xyz=0 0 0 rpy=0 0 0
- joint Shoulder_Pitch: limit lower=-1 upper=3 effort=0 velocity=0 -> lower=-1 upper=3 effort=100 velocity=100
