Commit message: moveit separated and fixed

File: config/so_100_arm.urdf.xacro (robot description, xacro)
@@ -3,5 +3,5 @@
     <xacro:arg name="initial_positions_file" default="initial_positions.yaml" />
     <!-- Import so_100_arm urdf file -->
-    <xacro:include filename="$(find so_100_arm)/urdf/so_100_arm_5dof.urdf" />
+    <xacro:include filename="$(find so_100_arm)/urdf/so_100_arm.urdf" />
     <!-- Import control_xacro -->
     <xacro:include filename="so_100_arm.ros2_control.xacro" />

File: urdf/so_100_arm.urdf (robot description, URDF)
Before this commit: robot so_100_arm, 9 links, 8 joints
Links:
- link Base: mass 0.146962928243327 -> 0.193184127927598
- link Fixed_Gripper: mass 0.11710741874408 -> 0.0929859131176897
- link Lower_Arm: mass 0.142523221917339 -> 0.147967774582291
- link Moving_Jaw: mass 0.0347149174448153 -> 0.0202443794940372
- link Shoulder_Rotation_Pitch: mass 0.111780100254674 -> 0.119226314127197
- link Upper_Arm: mass 0.167601391353176 -> 0.162409284599177
- link Wrist_Pitch_Roll: mass 0.106401896179987 -> 0.066132067097723
Joints:
- joint Elbow: axis 0 0 1 -> 1 0 0; origin xyz=-0.11238 0.0282 0 rpy=0 0 -2.2391 -> xyz=0 0.11257 0.028 rpy=0 0 0
- joint Gripper: origin xyz=0.0202 0 0.024375 rpy=-1.5708 0 0 -> xyz=-0.0202 -0.0244 0 rpy=3.1416 0 3.1416
- joint Shoulder_Pitch: axis 0 0 1 -> 1 0 0; origin xyz=0.000125 0.1086 0 rpy=3.1416 0 -1.5708 -> xyz=0 0.1025 0.0306 rpy=0 0 0
- joint Shoulder_Rotation: origin xyz=0 -0.0452 0.0181 rpy=1.5708 0 1.5708 -> xyz=0 -0.0452 0.0165 rpy=1.5708 0 0
- joint Wrist_Pitch: origin xyz=-0.1102 0.005375 0 rpy=0.90254 1.5708 0 -> xyz=0 0.0052 0.1349 rpy=0 0 0
- joint Wrist_Roll: axis 0 0 1 -> 0 1 0; origin xyz=0 0.002 -0.0545 rpy=3.1416 0 3.1416 -> xyz=0 -0.0601 0 rpy=0 0 0

Commit message: removed hardcoded path

File: config/so_100_arm.urdf.xacro (robot description, xacro)
@@ -3,5 +3,5 @@
     <xacro:arg name="initial_positions_file" default="initial_positions.yaml" />
     <!-- Import so_100_arm urdf file -->
-    <xacro:include filename="$(find so_100_arm)/urdf/so_100_arm.urdf" />
+    <xacro:include filename="$(find so_100_arm)/urdf/so_100_arm_5dof_hardware.urdf" />
     <!-- Import control_xacro -->
     <xacro:include filename="so_100_arm.ros2_control.xacro" />

File: urdf/so_100_arm.urdf (robot description, URDF)
Before this commit: robot so_100_arm, 9 links, 8 joints
Links:
- removed link world
Joints:
- removed joint world_to_base

File: urdf/so_100_arm_5dof.urdf (robot description, URDF)
Before this commit: robot so_100_arm, 9 links, 8 joints
Links:
- removed link world
Joints:
- removed joint world_to_base

File: urdf/so_100_arm_5dof_hardware.urdf (robot description, URDF)
Before this commit: robot so_100_arm, 9 links, 8 joints
Links:
- removed link world
Joints:
- removed joint world_to_base
- joint Elbow: origin xyz=0 0.11257 0.028 rpy=0 0 0 -> xyz=0 0.11257 0.028 rpy=-0.301 0 0
- joint Gripper: origin xyz=-0.0202 -0.0244 0 rpy=3.1416 0 3.1416 -> xyz=-0.0202 -0.0244 0 rpy=3.1416 0 2.8416
- joint Shoulder_Pitch: origin xyz=0 0.1025 0.0306 rpy=0 0 0 -> xyz=0 0.1025 0.0306 rpy=0.155 0 0
- joint Shoulder_Rotation: axis 0 1 0 -> 0 -1 0; origin xyz=0 -0.0452 0.0165 rpy=1.5708 0 0 -> xyz=0 -0.0452 0.0165 rpy=1.5708 0 -0.6
- joint Wrist_Pitch: origin xyz=0 0.0052 0.1349 rpy=0.707 0 0 -> xyz=0 0.0052 0.1349 rpy=-1.802 0 0
- joint Wrist_Roll: origin xyz=0 -0.0601 0 rpy=0 0 0 -> xyz=0 -0.0601 0 rpy=0 1.05708 0
