Commit message: moveit working

File: config/so_100_arm.ros2_control.xacro (robot description, xacro)
@@ -43,4 +43,11 @@
                 <state_interface name="velocity"/>
             </joint>
+            <joint name="Gripper">
+                <command_interface name="position"/>
+                <state_interface name="position">
+                    <param name="initial_value">0</param>
+                </state_interface>
+                <state_interface name="velocity"/>
+            </joint>
         </ros2_control>
     </xacro:macro>

Commit message: moveit joint limit added

File: config/so_100_arm.ros2_control.xacro (robot description, xacro)
@@ -2,5 +2,5 @@
 <robot xmlns:xacro="http://www.ros.org/wiki/xacro">
     <xacro:macro name="so_100_arm_ros2_control" params="name initial_positions_file">
-        <xacro:property name="initial_positions" value="${load_yaml(initial_positions_file)['initial_positions']}"/>
+        <xacro:property name="initial_positions" value="${xacro.load_yaml(initial_positions_file)['initial_positions']}"/>
         <ros2_control name="${name}" type="system">
             <hardware>
@@ -46,5 +46,5 @@
                 <command_interface name="position"/>
                 <state_interface name="position">
-                    <param name="initial_value">0</param>
+                  <param name="initial_value">${initial_positions['Gripper']}</param>
                 </state_interface>
                 <state_interface name="velocity"/>

Commit message: xacro arg added to launch real or mock arm

File: config/so_100_arm.ros2_control.xacro (robot description, xacro)
@@ -1,14 +1,17 @@
 <?xml version="1.0"?>
 <robot xmlns:xacro="http://www.ros.org/wiki/xacro">
-    <xacro:macro name="so_100_arm_ros2_control" params="name initial_positions_file">
+    <xacro:macro name="so_100_arm_ros2_control" params="name initial_positions_file use_fake_hardware" >
         <xacro:property name="initial_positions" value="${xacro.load_yaml(initial_positions_file)['initial_positions']}"/>
         <ros2_control name="${name}" type="system">
             <hardware>
-                <!-- By default, set up controllers for simulation. This won't work on real hardware -->
-                <!-- <plugin>mock_components/GenericSystem</plugin> -->
-                <plugin>so_arm_100_controller/SOARM100Interface</plugin>
-                <param name="use_serial">true</param>
-                <param name="serial_port">/dev/ttyUSB0</param>
-                <param name="serial_baudrate">1000000</param>
+                <xacro:if value="${use_fake_hardware}">
+                    <plugin>mock_components/GenericSystem</plugin>
+                </xacro:if>
+                <xacro:unless value="${use_fake_hardware}">
+                    <plugin>so_arm_100_controller/SOARM100Interface</plugin>
+                    <param name="use_serial">true</param>
+                    <param name="serial_port">/dev/ttyUSB0</param>
+                    <param name="serial_baudrate">1000000</param>
+                </xacro:unless>
             </hardware>
             <joint name="Shoulder_Rotation">

File: config/so_100_arm.urdf.xacro (robot description, xacro)
@@ -2,8 +2,12 @@
 <robot xmlns:xacro="http://www.ros.org/wiki/xacro" name="so_100_arm">
     <xacro:arg name="initial_positions_file" default="initial_positions.yaml" />
+    <xacro:arg name="use_fake_hardware" default="false"/>
     <!-- Import so_100_arm urdf file -->
     <xacro:include filename="$(find so_100_arm)/urdf/so_100_arm_5dof_hardware.urdf" />
     <!-- Import control_xacro -->
     <xacro:include filename="so_100_arm.ros2_control.xacro" />
-    <xacro:so_100_arm_ros2_control name="FakeSystem" initial_positions_file="$(arg initial_positions_file)"/>
+    <xacro:so_100_arm_ros2_control
+        name="SO100ARM"
+        initial_positions_file="$(arg initial_positions_file)"
+        use_fake_hardware="$(arg use_fake_hardware)"/>
 </robot>
